File: hardware/arduino-micro/arduino-micro.sch (KiCad schematic (older format))
At the start: 9 parts, among them J1 PJ-028-SMT-TR, M1 Fan_4pin, SW1 Rotary_Encoder, U1 TM1637, U2 CA56-12CGKWA

Commit message: fixes for cnc'd pcb
Parts:
- added C1: 100uF, Capacitor_THT:CP_Radial_Tantal_D4.5mm_P2.50mm, symbol Device:CP
- added C2: 0.1uF, Capacitor_SMD:C_0805_2012Metric, symbol Device:C
- added C3, C4: 100pF, Capacitor_SMD:C_0805_2012Metric, symbol Device:C
- added R4, R5: 10k, Resistor_SMD:R_0805_2012Metric, symbol Device:R
- R1, R2, R3: footprint LED_SMD:LED_0805_2012Metric -> Resistor_SMD:R_0805_2012Metric
Connections:
- wire segments 91 -> 113
Changed lines of the file:
@@
 F 0 "R3" H 10230 4654 50  0000 R CNN
 F 1 "10k" H 10230 4745 50  0000 R CNN
-F 2 "LED_SMD:LED_0805_2012Metric" V 10230 4700 50  0001 C CNN
+F 2 "Resistor_SMD:R_0805_2012Metric" V 10230 4700 50  0001 C CNN
 F 3 "~" H 10300 4700 50  0001 C CNN
 	1    10300 4700
@@
 F 0 "R1" V 5893 4300 50  0000 C CNN
 F 1 "10k" V 5984 4300 50  0000 C CNN
-F 2 "LED_SMD:LED_0805_2012Metric" V 6030 4300 50  0001 C CNN
+F 2 "Resistor_SMD:R_0805_2012Metric" V 6030 4300 50  0001 C CNN
 F 3 "~" H 6100 4300 50  0001 C CNN
 	1    6100 4300
@@
 F 0 "R2" V 5893 4500 50  0000 C CNN
 F 1 "10k" V 5984 4500 50  0000 C CNN
-F 2 "LED_SMD:LED_0805_2012Metric" V 6030 4500 50  0001 C CNN
+F 2 "Resistor_SMD:R_0805_2012Metric" V 6030 4500 50  0001 C CNN
 F 3 "~" H 6100 4500 50  0001 C CNN
 	1    6100 4500
@@
 	1    0    0    -1
 $EndComp
-Wire Wire Line
-	3200 1950 3400 1950
-Wire Wire Line
-	3200 2050 3400 2050
-Wire Wire Line
-	3200 2150 3400 2150
-Text Label 3400 1950 0    50   ~ 0
+Text Label 4650 1950 0    50   ~ 0
 7S_CLK
-Text Label 3400 2050 0    50   ~ 0
+Text Label 4650 2050 0    50   ~ 0
 7S_IO
-Text Label 3400 2150 0    50   ~ 0
+Text Label 2200 950  2    50   ~ 0
 5V
-Wire Wire Line
-	2300 1750 2100 1750
-Text Label 2100 1750 2    50   ~ 0
-VSS
 Wire Wire Line
 	9450 3950 9550 3950
@@
 	5700 5650 5900 5650
 Connection ~ 5900 5650
+$Comp
+L Device:R R5
+U 1 1 5BD62940
+P 4450 1550
+F 0 "R5" H 4520 1596 50  0000 L CNN
+F 1 "10k" H 4520 1505 50  0000 L CNN
+F 2 "Resistor_SMD:R_0805_2012Metric" V 4380 1550 50  0001 C CNN
+F 3 "~" H 4450 1550 50  0001 C CNN
+	1    4450 1550
+	1    0    0    -1
+$EndComp
+$Comp
+L Device:R R4
+U 1 1 5BD6582F
+P 4150 1550
+F 0 "R4" H 4220 1596 50  0000 L CNN
+F 1 "10k" H 4220 1505 50  0000 L CNN
+F 2 "Resistor_SMD:R_0805_2012Metric" V 4080 1550 50  0001 C CNN
+F 3 "~" H 4150 1550 50  0001 C CNN
+	1    4150 1550
+	1    0    0    -1
+$EndComp
+$Comp
+L Device:C C4
+U 1 1 5BD688AC
+P 3750 1550
+F 0 "C4" H 3865 1596 50  0000 L CNN
+F 1 "100pF" H 3865 1505 50  0000 L CNN
+F 2 "Capacitor_SMD:C_0805_2012Metric" H 3788 1400 50  0001 C CNN
+F 3 "~" H 3750 1550 50  0001 C CNN
+	1    3750 1550
+	1    0    0    -1
+$EndComp
+Wire Wire Line
+	3200 1950 3750 1950
+$Comp
+L Device:C C3
+U 1 1 5BD7521D
+P 3450 1550
+F 0 "C3" H 3565 1596 50  0000 L CNN
+F 1 "100pF" H 3565 1505 50  0000 L CNN
+F 2 "Capacitor_SMD:C_0805_2012Metric" H 3488 1400 50  0001 C CNN
+F 3 "~" H 3450 1550 50  0001 C CNN
+	1    3450 1550
+	1    0    0    -1
+$EndComp
+Wire Wire Line
+	4150 1700 4150 2050
+Connection ~ 4150 2050
+Wire Wire Line
+	4150 2050 4650 2050
+Wire Wire Line
+	4450 1700 4450 1950
+Connection ~ 4450 1950
+Wire Wire Line
+	4450 1950 4650 1950
+Wire Wire Line
+	3750 1700 3750 1950
+Connection ~ 3750 1950
+Wire Wire Line
+	3750 1950 4450 1950
+$Comp
+L Device:CP C1
+U 1 1 5BD84599
+P 2500 1100
+F 0 "C1" H 2618 1146 50  0000 L CNN
+F 1 "100uF" H 2618 1055 50  0000 L CNN
+F 2 "Capacitor_THT:CP_Radial_Tantal_D4.5mm_P2.50mm" H 2538 950 50  0001 C CNN
+F 3 "~" H 2500 1100 50  0001 C CNN
+	1    2500 1100
+	1    0    0    -1
+$EndComp
+$Comp
+L Device:C C2
+U 1 1 5BD8E2D1
+P 3000 1100
+F 0 "C2" H 3115 1146 50  0000 L CNN
+F 1 "0.1uF" H 3115 1055 50  0000 L CNN
+F 2 "Capacitor_SMD:C_0805_2012Metric" H 3038 950 50  0001 C CNN
+F 3 "~" H 3000 1100 50  0001 C CNN
+	1    3000 1100
+	1    0    0    -1
+$EndComp
+Wire Wire Line
+	2200 950  2500 950
+Wire Wire Line
+	3000 950  3300 950
+Wire Wire Line
+	3300 950  3300 2150
+Wire Wire Line
+	3300 2150 3200 2150
+Connection ~ 3000 950
+Wire Wire Line
+	2300 1250 2300 1750
+Wire Wire Line
+	3200 2050 3450 2050
+Wire Wire Line
+	3450 1700 3450 2050
+Connection ~ 3450 2050
+Wire Wire Line
+	3450 2050 4150 2050
+Wire Wire Line
+	3600 1250 3600 1400
+Wire Wire Line
+	3600 1400 3750 1400
+Wire Wire Line
+	3600 1400 3450 1400
+Connection ~ 3600 1400
+Wire Wire Line
+	3600 1250 3000 1250
+Connection ~ 3000 1250
+Text Label 3750 1250 0    50   ~ 0
+VSS
+Wire Wire Line
+	3600 1250 3750 1250
+Connection ~ 3600 1250
+Connection ~ 2500 950
+Connection ~ 2500 1250
+Wire Wire Line
+	2500 1250 2300 1250
+Wire Wire Line
+	2500 950  3000 950
+Wire Wire Line
+	2500 1250 3000 1250
+Wire Wire Line
+	4150 1400 4300 1400
+Wire Wire Line
+	4300 1400 4300 1250
+Connection ~ 4300 1400
+Wire Wire Line
+	4300 1400 4450 1400
+Text Label 4300 1250 0    50   ~ 0
+5V
 $EndSCHEMATC

Commit message: Ch ch ch changes.
Parts:
- added R6: 27k, coddingtonbear:0805_Milling, symbol pspice:R
- added R7: 10k, coddingtonbear:0805_Milling, symbol pspice:R
- C1: footprint Capacitor_THT:CP_Radial_Tantal_D4.5mm_P2.50mm -> Capacitors_THT:CP_Radial_D6.3mm_P2.50mm; symbol Device:CP -> arduino-micro-rescue:CP-Device
- C2, C3, C4: footprint Capacitor_SMD:C_0805_2012Metric -> coddingtonbear:0805_Milling; symbol Device:C -> arduino-micro-rescue:C-Device
- M1: symbol Motor:Fan_4pin -> arduino-micro-rescue:Fan_4pin-Motor
- R1, R2, R3, R4, R5: footprint Resistor_SMD:R_0805_2012Metric -> coddingtonbear:0805_Milling; symbol Device:R -> arduino-micro-rescue:R-Device
- SW1: symbol Device:Rotary_Encoder -> arduino-micro-rescue:Rotary_Encoder-Device
- U2: symbol Display_Character:CA56-12CGKWA -> arduino-micro-rescue:CA56-12CGKWA-Display_Character
Changed lines of the file:
@@
 $EndDescr
-$Comp
-L arduino:Arduino_Micro_Socket XA1
-U 1 1 5BCC7897
-P 8150 4050
-F 0 "XA1" H 8150 5287 60  0000 C CNN
-F 1 "Arduino_Micro_Socket" H 8150 5181 60  0000 C CNN
-F 2 "Arduino:Arduino_Micro_Socket" H 9950 7800 60  0001 C CNN
-F 3 "https://store.arduino.cc/arduino-micro" H 9950 7800 60  0001 C CNN
-	1    8150 4050
-	1    0    0    -1
-$EndComp
 $Comp
 L PJ-028-SMT-TR:PJ-028-SMT-TR J1
@@
 $EndComp
 $Comp
-L Motor:Fan_4pin M1
+L arduino-micro-rescue:Fan_4pin-Motor M1
 U 1 1 5BCC886A
 P 10450 5300
@@
 	10050 3250 9450 3250
 $Comp
-L Device:R R3
+L arduino-micro-rescue:R-Device R3
 U 1 1 5BCCBA37
 P 10300 4700
 F 0 "R3" H 10230 4654 50  0000 R CNN
 F 1 "10k" H 10230 4745 50  0000 R CNN
-F 2 "Resistor_SMD:R_0805_2012Metric" V 10230 4700 50  0001 C CNN
+F 2 "coddingtonbear:0805_Milling" V 10230 4700 50  0001 C CNN
 F 3 "~" H 10300 4700 50  0001 C CNN
 	1    10300 4700
@@
 	10300 5000 9650 5000
 $Comp
-L Device:Rotary_Encoder SW1
+L arduino-micro-rescue:Rotary_Encoder-Device SW1
 U 1 1 5BCCC134
 P 5250 4050
@@
 	6450 4250 6850 4250
 $Comp
-L Device:R R1
+L arduino-micro-rescue:R-Device R1
 U 1 1 5BCCD0CA
 P 6100 4300
 F 0 "R1" V 5893 4300 50  0000 C CNN
 F 1 "10k" V 5984 4300 50  0000 C CNN
-F 2 "Resistor_SMD:R_0805_2012Metric" V 6030 4300 50  0001 C CNN
+F 2 "coddingtonbear:0805_Milling" V 6030 4300 50  0001 C CNN
 F 3 "~" H 6100 4300 50  0001 C CNN
 	1    6100 4300
@@
 $EndComp
 $Comp
-L Device:R R2
+L arduino-micro-rescue:R-Device R2
 U 1 1 5BCCD17E
 P 6100 4500
 F 0 "R2" V 5893 4500 50  0000 C CNN
 F 1 "10k" V 5984 4500 50  0000 C CNN
-F 2 "Resistor_SMD:R_0805_2012Metric" V 6030 4500 50  0001 C CNN
+F 2 "coddingtonbear:0805_Milling" V 6030 4500 50  0001 C CNN
 F 3 "~" H 6100 4500 50  0001 C CNN
 	1    6100 4500
@@
 Text Label 6350 4850 0    50   ~ 0
 5V
-Wire Wire Line
-	10150 4400 10150 3450
-Wire Wire Line
-	10150 3450 9450 3450
-Connection ~ 10150 4400
 $Comp
 L squeeze-misc:TM1637 U1
@@
 Text Label 2200 950  2    50   ~ 0
 5V
-Wire Wire Line
-	9450 3950 9550 3950
-Text Label 9550 3950 0    50   ~ 0
+Text Label 9450 4450 0    50   ~ 0
 7S_CLK
-Wire Wire Line
-	9450 4050 9550 4050
-Text Label 9550 4050 0    50   ~ 0
+Text Label 9450 4350 0    50   ~ 0
 7S_IO
 $Comp
-L Display_Character:CA56-12CGKWA U2
+L arduino-micro-rescue:CA56-12CGKWA-Display_Character U2
 U 1 1 5BCDF577
 P 2850 3700
@@
 NoConn ~ 9450 3850
 NoConn ~ 9450 4250
-NoConn ~ 9450 4350
-NoConn ~ 9450 4450
 NoConn ~ 9450 4550
 NoConn ~ 9450 4750
@@
 Connection ~ 5900 5650
 $Comp
-L Device:R R5
+L arduino-micro-rescue:R-Device R5
 U 1 1 5BD62940
 P 4450 1550
 F 0 "R5" H 4520 1596 50  0000 L CNN
 F 1 "10k" H 4520 1505 50  0000 L CNN
-F 2 "Resistor_SMD:R_0805_2012Metric" V 4380 1550 50  0001 C CNN
+F 2 "coddingtonbear:0805_Milling" V 4380 1550 50  0001 C CNN
 F 3 "~" H 4450 1550 50  0001 C CNN
 	1    4450 1550
@@
 $EndComp
 $Comp
-L Device:R R4
+L arduino-micro-rescue:R-Device R4
 U 1 1 5BD6582F
 P 4150 1550
 F 0 "R4" H 4220 1596 50  0000 L CNN
 F 1 "10k" H 4220 1505 50  0000 L CNN
-F 2 "Resistor_SMD:R_0805_2012Metric" V 4080 1550 50  0001 C CNN
+F 2 "coddingtonbear:0805_Milling" V 4080 1550 50  0001 C CNN
 F 3 "~" H 4150 1550 50  0001 C CNN
 	1    4150 1550
@@
 $EndComp
 $Comp
-L Device:C C4
+L arduino-micro-rescue:C-Device C4
 U 1 1 5BD688AC
 P 3750 1550
 F 0 "C4" H 3865 1596 50  0000 L CNN
 F 1 "100pF" H 3865 1505 50  0000 L CNN
-F 2 "Capacitor_SMD:C_0805_2012Metric" H 3788 1400 50  0001 C CNN
+F 2 "coddingtonbear:0805_Milling" H 3788 1400 50  0001 C CNN
 F 3 "~" H 3750 1550 50  0001 C CNN
 	1    3750 1550
@@
 	3200 1950 3750 1950
 $Comp
-L Device:C C3
+L arduino-micro-rescue:C-Device C3
 U 1 1 5BD7521D
 P 3450 1550
 F 0 "C3" H 3565 1596 50  0000 L CNN
 F 1 "100pF" H 3565 1505 50  0000 L CNN
-F 2 "Capacitor_SMD:C_0805_2012Metric" H 3488 1400 50  0001 C CNN
+F 2 "coddingtonbear:0805_Milling" H 3488 1400 50  0001 C CNN
 F 3 "~" H 3450 1550 50  0001 C CNN
 	1    3450 1550
@@
 	3750 1950 4450 1950
 $Comp
-L Device:CP C1
+L arduino-micro-rescue:CP-Device C1
 U 1 1 5BD84599
 P 2500 1100
 F 0 "C1" H 2618 1146 50  0000 L CNN
 F 1 "100uF" H 2618 1055 50  0000 L CNN
-F 2 "Capacitor_THT:CP_Radial_Tantal_D4.5mm_P2.50mm" H 2538 950 50  0001 C CNN
+F 2 "Capacitors_THT:CP_Radial_D6.3mm_P2.50mm" H 2538 950 50  0001 C CNN
 F 3 "~" H 2500 1100 50  0001 C CNN
 	1    2500 1100
@@
 $EndComp
 $Comp
-L Device:C C2
+L arduino-micro-rescue:C-Device C2
 U 1 1 5BD8E2D1
 P 3000 1100
 F 0 "C2" H 3115 1146 50  0000 L CNN
 F 1 "0.1uF" H 3115 1055 50  0000 L CNN
-F 2 "Capacitor_SMD:C_0805_2012Metric" H 3038 950 50  0001 C CNN
+F 2 "coddingtonbear:0805_Milling" H 3038 950 50  0001 C CNN
 F 3 "~" H 3000 1100 50  0001 C CNN
 	1    3000 1100
@@
 Text Label 4300 1250 0    50   ~ 0
 5V
+$Comp
+L pspice:R R6
+U 1 1 5BE18F60
+P 10150 3850
+F 0 "R6" H 10218 3896 50  0000 L CNN
+F 1 "27k" H 10218 3805 50  0000 L CNN
+F 2 "coddingtonbear:0805_Milling" H 10150 3850 50  0001 C CNN
+F 3 "~" H 10150 3850 50  0001 C CNN
+	1    10150 3850
+	1    0    0    -1
+$EndComp
+$Comp
+L pspice:R R7
+U 1 1 5BE18FDD
+P 10500 3450
+F 0 "R7" V 10295 3450 50  0000 C CNN
+F 1 "10k" V 10386 3450 50  0000 C CNN
+F 2 "coddingtonbear:0805_Milling" H 10500 3450 50  0001 C CNN
+F 3 "~" H 10500 3450 50  0001 C CNN
+	1    10500 3450
+	0    1    1    0
+$EndComp
+Wire Wire Line
+	10150 4400 10150 4100
+Connection ~ 10150 4400
+Wire Wire Line
+	10150 3600 10150 3450
+Wire Wire Line
+	10150 3450 9450 3450
+Wire Wire Line
+	10250 3450 10150 3450
+Connection ~ 10150 3450
+$Comp
+L power:GND #PWR0103
+U 1 1 5BE2E5E8
+P 10750 3450
+F 0 "#PWR0103" H 10750 3200 50  0001 C CNN
+F 1 "GND" H 10755 3277 50  0000 C CNN
+F 2 "" H 10750 3450 50  0001 C CNN
+F 3 "" H 10750 3450 50  0001 C CNN
+	1    10750 3450
+	1    0    0    -1
+$EndComp
+$Comp
+L arduino:Arduino_Micro_Socket XA1
+U 1 1 5BCC7897
+P 8150 4050
+F 0 "XA1" H 8150 5287 60  0000 C CNN
+F 1 "Arduino_Micro_Socket" H 8150 5181 60  0000 C CNN
+F 2 "Arduino:Arduino_Micro_Socket" H 9950 7800 60  0001 C CNN
+F 3 "https://store.arduino.cc/arduino-micro" H 9950 7800 60  0001 C CNN
+	1    8150 4050
+	1    0    0    -1
+$EndComp
+NoConn ~ 9450 3950
+NoConn ~ 9450 4050
 $EndSCHEMATC
