File: hardware/arduino-micro/arduino-micro.sch (KiCad schematic (older format))
At the start: 24 parts, among them J1 PJ-088CH, J2 i2c_header, M1 Fan_4pin, SW1 Rotary_Encoder, U1 TM1637, U2 CA56-12CGKWA, U3 BUTTON_1, U4 BUTTON_2, U5 BUTTON_3

Commit message: board updates for prototype
Parts:
- J1: value PJ-088CH -> PJ-083H; footprint PJ-088CH:CUI_PJ-088CH -> squeeze-misc:CUI_PJ-083H; symbol PJ-088CH:PJ-088CH -> PJ-083H:PJ-083H
Connections:
- net GND: now also J1.3; no longer J1.3.1 (3), J1.3.2 (3)
- new net: J1.S1 (SHIELD), J1.S2 (SHIELD)
- no-connect marks 23 -> 24
Changed lines of the file:
@@
 	5700 5650 5900 5650
-Wire Wire Line
-	5450 5450 6100 5450
-$Comp
-L PJ-088CH:PJ-088CH J1
-U 1 1 5D8F4C7C
-P 5150 5350
-F 0 "J1" H 5195 5690 50  0000 C CNN
-F 1 "PJ-088CH" H 5195 5599 50  0000 C CNN
-F 2 "PJ-088CH:CUI_PJ-088CH" H 5150 5350 50  0001 L BNN
-F 3 "1.0" H 5150 5350 50  0001 L BNN
-F 4 "CUI" H 5150 5350 50  0001 L BNN "Field4"
-F 5 "Manufacturer Recommendations" H 5150 5350 50  0001 L BNN "Field5"
-	1    5150 5350
-	1    0    0    -1
-$EndComp
 Wire Wire Line
 	5450 5350 6100 5350
@@
 Wire Wire Line
 	5750 3000 5850 3000
+$Comp
+L PJ-083H:PJ-083H J1
+U 1 1 5D8F4C7C
+P 4950 5450
+F 0 "J1" H 4950 5900 50  0000 C CNN
+F 1 "PJ-083H" H 4950 5800 50  0000 C CNN
+F 2 "squeeze-misc:CUI_PJ-083H" H 4950 5450 50  0001 L BNN
+F 3 "1.0" H 4950 5450 50  0001 L BNN
+F 4 "CUI" H 4950 5450 50  0001 L BNN "Field4"
+F 5 "Manufacturer Recommendations" H 4950 5450 50  0001 L BNN "Field5"
+	1    4950 5450
+	1    0    0    -1
+$EndComp
+Wire Wire Line
+	5450 5450 6100 5450
+NoConn ~ 5450 5650
 $EndSCHEMATC
